Commit message: added approximate coefficients

File: urdf/noir_description/urdf/noir.xacro (robot description, xacro)
@@ -9,6 +9,6 @@
   <xacro:property name="mass" value="5" /> <!-- [kg] -->
   <xacro:property name="body_width" value="1.05" /> <!-- [m] -->
-  <xacro:property name="body_height" value="0.11" /> <!-- [m] -->
-  <xacro:property name="mass_rotor" value="0.005" /> <!-- [kg] -->
+  <xacro:property name="body_height" value="0.14" /> <!-- [m] -->
+  <xacro:property name="mass_rotor" value="0.05" /> <!-- [kg] -->
   <xacro:property name="arm_length_front_x" value="0.265" /> <!-- [m] -->
   <xacro:property name="arm_length_back_x" value="0.265" /> <!-- [m] -->
@@ -17,9 +17,9 @@
   <xacro:property name="rotor_offset_top" value="0.078" /> <!-- [m] -->
   <xacro:property name="radius_rotor" value="0.2286" /> <!-- [m] -->
-  <xacro:property name="motor_constant" value="8.54858e-06" /> <!-- [kg.m/s^2] -->
-  <xacro:property name="moment_constant" value="0.06" /> <!-- [m] -->
-  <xacro:property name="time_constant_up" value="0.0125" /> <!-- [s] -->
-  <xacro:property name="time_constant_down" value="0.025" /> <!-- [s] -->
-  <xacro:property name="max_rot_velocity" value="1100" /> <!-- [rad/s] -->
+  <xacro:property name="motor_constant" value="0.00007974352" /> <!-- [kg.m/s^2] -->
+  <xacro:property name="moment_constant" value="0.02893726238" /> <!-- [m] -->
+  <xacro:property name="time_constant_up" value="0.025" /> <!-- [s] -->
+  <xacro:property name="time_constant_down" value="0.05" /> <!-- [s] -->
+  <xacro:property name="max_rot_velocity" value="565.486677646" /> <!-- [rad/s] -->
   <xacro:property name="sin30" value="0.5" />
   <xacro:property name="cos30" value="0.866025403784" />
