Commit message: compiled urdf and added launch file

File: urdf/noir_description/urdf/multirotor_base.xacro (robot description, xacro)
@@ -96,5 +96,5 @@
           <!-- <cylinder length="0.005" radius="${radius_rotor}"/> --> <!-- [m] -->
           <!-- <mesh filename="package://rotors_description/meshes/propeller_${direction}.dae" -->
-          <mesh filename="package://rotors_description/meshes/${mesh}_${direction}.dae"
+          <mesh filename="package://rotors_description/meshes/${mesh}.stl"
             scale="${mesh_scale}" />
           <!-- <box size="${2*radius_rotor} 0.01 0.005"/> -->

File: urdf/noir_description/urdf/noir.xacro (robot description, xacro)
@@ -5,4 +5,5 @@
   <xacro:property name="rotor_velocity_slowdown_sim" value="10" />
   <xacro:property name="mesh_file" value="CF_assembly.stl" />
+  <xacro:property name="prop_mesh" value="prop18" />
   <xacro:property name="mesh_scale" value="1 1 1"/>
   <xacro:property name="mesh_scale_prop" value="1 1 1"/>
@@ -70,5 +71,5 @@
     rotor_drag_coefficient="${rotor_drag_coefficient}"
     rolling_moment_coefficient="${rolling_moment_coefficient}"
-    mesh="noir_prop"
+    mesh="${prop_mesh}"
     mesh_scale="${mesh_scale_prop}"
     color="Blue">
@@ -91,5 +92,5 @@
     rotor_drag_coefficient="${rotor_drag_coefficient}"
     rolling_moment_coefficient="${rolling_moment_coefficient}"
-    mesh="noir_prop"
+    mesh="${prop_mesh}"
     mesh_scale="${mesh_scale_prop}"
     color="DarkGrey">
@@ -111,5 +112,5 @@
     rotor_drag_coefficient="${rotor_drag_coefficient}"
     rolling_moment_coefficient="${rolling_moment_coefficient}"
-    mesh="noir_prop"
+    mesh="${prop_mesh}"
     mesh_scale="${mesh_scale_prop}"
     color="Blue">
@@ -131,5 +132,5 @@
     rotor_drag_coefficient="${rotor_drag_coefficient}"
     rolling_moment_coefficient="${rolling_moment_coefficient}"
-    mesh="noir_prop"
+    mesh="${prop_mesh}"
     mesh_scale="${mesh_scale_prop}"
     color="DarkGrey">

Commit message: issue getting stl rendering

File: urdf/noir_description/urdf/multirotor_base.xacro (robot description, xacro)
@@ -36,5 +36,5 @@
         <origin xyz="0 0 0" rpy="0 0 0" />
         <geometry>
-          <mesh filename="package://rotors_description/meshes/${mesh_file}"
+          <mesh filename="~/catkin_ws/src/mission7_master/urdf/noir_description/meshes/${mesh_file}"
             scale="${mesh_scale}" />
           <!-- <box size="${body_width} ${body_width} ${body_height}"/> --> <!-- [m] [m] [m] -->
@@ -96,5 +96,5 @@
           <!-- <cylinder length="0.005" radius="${radius_rotor}"/> --> <!-- [m] -->
           <!-- <mesh filename="package://rotors_description/meshes/propeller_${direction}.dae" -->
-          <mesh filename="package://rotors_description/meshes/${mesh}.stl"
+          <mesh filename="~/catkin_ws/src/mission7_master/urdf/noir_description/meshes/${mesh}.stl"
             scale="${mesh_scale}" />
           <!-- <box size="${2*radius_rotor} 0.01 0.005"/> -->

Commit message: got model to render

File: urdf/noir_description/urdf/multirotor_base.xacro (robot description, xacro)
@@ -36,5 +36,5 @@
         <origin xyz="0 0 0" rpy="0 0 0" />
         <geometry>
-          <mesh filename="~/catkin_ws/src/mission7_master/urdf/noir_description/meshes/${mesh_file}"
+          <mesh filename="model://noir_description/meshes/${mesh_file}"
             scale="${mesh_scale}" />
           <!-- <box size="${body_width} ${body_width} ${body_height}"/> --> <!-- [m] [m] [m] -->
@@ -96,5 +96,5 @@
           <!-- <cylinder length="0.005" radius="${radius_rotor}"/> --> <!-- [m] -->
           <!-- <mesh filename="package://rotors_description/meshes/propeller_${direction}.dae" -->
-          <mesh filename="~/catkin_ws/src/mission7_master/urdf/noir_description/meshes/${mesh}.stl"
+          <mesh filename="model://noir_description/meshes/${mesh}.stl"
             scale="${mesh_scale}" />
           <!-- <box size="${2*radius_rotor} 0.01 0.005"/> -->
