Commit message: added stereo cameras to simulation

File: robot_description/noir_description/urdf/component_snippets.xacro (robot description, xacro)
@@ -32,4 +32,84 @@
     </gazebo>
   </xacro:macro>
+<!-- Macro to add a stereo camera -->
+<xacro:macro name="stereo_camera_macro" params="namespace parent_link camera_suffix base_line enable_visual *cylinder *origin">
+<link name="${namespace}/camera_${camera_suffix}_link">
+      <collision>
+        <origin xyz="0 0 0" rpy="0 0 0" />
+        <geometry>
+          <xacro:insert_block name="cylinder" />
+        </geometry>
+      </collision>
+      <xacro:if value="${enable_visual}">
+        <visual>
+          <origin xyz="0 0 0" rpy="0 1.57079632679 0" />
+          <geometry>
+            <xacro:insert_block name="cylinder" />
+          </geometry>
+          <material name="red" />
+        </visual>
+      </xacro:if>
+      <inertial>
+        <mass value="1e-5" />
+        <origin xyz="0 0 0" rpy="0 0 0" />
+        <inertia ixx="1e-6" ixy="0" ixz="0" iyy="1e-6" iyz="0" izz="1e-6" />
+      </inertial>
+    </link>
+    <joint name="${namespace}/camera_${camera_suffix}_joint" type="fixed">
+      <xacro:insert_block name="origin" />
+      <parent link="${parent_link}" />
+      <child link="${namespace}/camera_${camera_suffix}_link" />
+    </joint>
+<gazebo reference="${namespace}/camera_${camera_suffix}_link">
+    <sensor type="multicamera" name="stereo_camera">
+      <!-- see MultiSenseSLPlugin.h for available modes -->
+      <update_rate>30.0</update_rate>
+      <camera name="left">
+	<!-- Spec sheet says 80deg X 45deg @ 1024x544pix.  Based on feedback
+	    from teams, we're instead doing 80deg X 80deg @ 800x800pix. -->
+	<horizontal_fov>1.3962634</horizontal_fov>
+	<image>
+	  <width>752</width>
+	  <height>480</height>
+	  <format>R8G8B8</format>
+	</image>
+	<clip>
+	  <near>0.02</near>
+	  <far>100</far>
+	</clip>
+      </camera>
+      <camera name="right">
+	<pose>0 -${base_line} 0 0 0 0</pose>
+	<!-- Spec sheet says 80deg X 45deg @ 1024x544pix.  Based on feedback
+	    from teams, we're instead doing 80deg X 80deg @ 800x800pix. -->
+	<horizontal_fov>1.3962634</horizontal_fov>
+	<image>
+	  <width>752</width>
+	  <height>480</height>
+	  <format>R8G8B8</format>
+	</image>
+	<clip>
+	  <near>0.02</near>
+	  <far>100</far>
+	</clip>
+      </camera>
+      <plugin name="stereo_camera_controller" filename="libgazebo_ros_multicamera.so">
+	<alwaysOn>true</alwaysOn>
+	<updateRate>0.0</updateRate>
+	<cameraName>camera_${camera_suffix}</cameraName>
+	<imageTopicName>image_raw</imageTopicName>
+	<cameraInfoTopicName>camera_info</cameraInfoTopicName>
+	<frameName>${namespace}/camera_${camera_suffix}_link</frameName>
+	<!--<rightFrameName>right_camera_optical_frame</rightFrameName>-->
+	<hackBaseline>${base_line}</hackBaseline>
+	<distortionK1>0.0</distortionK1>
+	<distortionK2>0.0</distortionK2>
+	<distortionK3>0.0</distortionK3>
+	<distortionT1>0.0</distortionT1>
+	<distortionT2>0.0</distortionT2>
+      </plugin>
+    </sensor>
+  </gazebo>
+</xacro:macro>
   <!-- Macro to add a camera. -->
   <xacro:macro name="camera_macro"
@@ -478,10 +558,10 @@
     </joint>
     <!-- Cameras -->
-    <xacro:if value="$(arg enable_cameras)">
+    <xacro:if value="true">
       <!-- Left Camera -->
       <xacro:vi_sensor_camera_macro
         namespace="${namespace}" parent_link="${namespace}/vi_sensor_link"
         camera_suffix="left" frame_rate="30.0">
-        <origin xyz="0.015 0.055 0.0065" rpy="0 0 0" />
+        <origin xyz="0.015 0.03805 0.0065" rpy="0 0 0" />
       </xacro:vi_sensor_camera_macro>
       <!-- Right Camera -->
@@ -489,9 +569,9 @@
         parent_link="${namespace}/vi_sensor_link"
         camera_suffix="right" frame_rate="30.0">
-        <origin xyz="0.015 -0.055 0.0065" rpy="0 0 0" />
+        <origin xyz="0.015 -0.03805 0.0065" rpy="0 0 0" />
       </xacro:vi_sensor_camera_macro>
     </xacro:if>
     <!-- Depth Sensor -->
-    <xacro:if value="$(arg enable_depth)">
+    <xacro:if value="false">
       <xacro:vi_sensor_depth_macro
         namespace="${namespace}" parent_link="${namespace}/vi_sensor_link"
@@ -501,5 +581,5 @@
     </xacro:if>
     <!-- Groundtruth -->
-    <xacro:if value="$(arg enable_ground_truth)">
+    <xacro:if value="false">
       <!-- Odometry Sensor -->
       <xacro:odometry_plugin_macro
@@ -533,9 +613,10 @@
     </xacro:if>
     <!-- ADIS16448 IMU. -->
+<xacro:if value="false">
     <xacro:imu_plugin_macro
       namespace="${namespace}"
       imu_suffix=""
       parent_link="${namespace}/vi_sensor_link"
-      imu_topic="/imu"
+      imu_topic="/imu_vi"
       mass_imu_sensor="0.015"
       gyroscope_noise_density="0.0003394"
@@ -550,4 +631,5 @@
       <origin xyz="0.015 0 0.0113" rpy="0 0 0" />
     </xacro:imu_plugin_macro>
+</xacro:if>
   </xacro:macro>
 </robot>

File: robot_description/noir_description/urdf/noir_base.xacro (robot description, xacro)
@@ -38,4 +38,19 @@
         />
   </xacro:if>
+<!--stereo camera-->
+<xacro:if value="true">
+<xacro:stereo_camera_macro
+    namespace="${namespace}"
+    camera_suffix="front"
+parent_link="base_link"
+base_line="0.076"
+enable_visual="true"
+    >
+<cylinder length="0.04" radius="0.04" />
+    <origin xyz="0 0 0.4" rpy="0 0 0" />
+</xacro:stereo_camera_macro>
+</xacro:if>
+<!--standard camera-->
+<xacro:if value="false">
 <xacro:camera_macro
     namespace="${namespace}"
@@ -56,6 +71,7 @@
     <origin xyz="0 0 0.4" rpy="0 0 0" />
 </xacro:camera_macro>
+</xacro:if>
     <!-- Instantiate gps plugin. -->
-<xacro:if value="true">
+<xacro:if value="false">
   <xacro:gps_plugin_macro
     namespace="${namespace}"

Commit message: put quad in iarc world

File: robot_description/noir_description/urdf/component_snippets.xacro (robot description, xacro)
@@ -34,5 +34,5 @@
 <!-- Macro to add a stereo camera -->
 <xacro:macro name="stereo_camera_macro" params="namespace parent_link camera_suffix base_line enable_visual *cylinder *origin">
-<link name="${namespace}/camera_${camera_suffix}_link">
+<link name="${namespace}/camera_${camera_suffix}_left_optical_link">
       <collision>
         <origin xyz="0 0 0" rpy="0 0 0" />
@@ -56,10 +56,37 @@
       </inertial>
     </link>
-    <joint name="${namespace}/camera_${camera_suffix}_joint" type="fixed">
+    <joint name="${namespace}/camera_${camera_suffix}_left_optical_joint" type="fixed">
       <xacro:insert_block name="origin" />
       <parent link="${parent_link}" />
-      <child link="${namespace}/camera_${camera_suffix}_link" />
-    </joint>
-<gazebo reference="${namespace}/camera_${camera_suffix}_link">
+      <child link="${namespace}/camera_${camera_suffix}_left_optical_link" />
+    </joint>
+<link name="${namespace}/camera_${camera_suffix}_right_optical_link">
+      <collision>
+        <origin xyz="0 0 0" rpy="0 0 0" />
+        <geometry>
+          <xacro:insert_block name="cylinder" />
+        </geometry>
+      </collision>
+      <xacro:if value="${enable_visual}">
+        <visual>
+          <origin xyz="0 0 0" rpy="0 1.57079632679 0" />
+          <geometry>
+            <xacro:insert_block name="cylinder" />
+          </geometry>
+          <material name="red" />
+        </visual>
+      </xacro:if>
+      <inertial>
+        <mass value="1e-5" />
+        <origin xyz="0 0 0" rpy="0 0 0" />
+        <inertia ixx="1e-6" ixy="0" ixz="0" iyy="1e-6" iyz="0" izz="1e-6" />
+      </inertial>
+    </link>
+    <joint name="${namespace}/camera_${camera_suffix}_right_optical_joint" type="fixed">
+      <origin xyz="0 -${base_line} 0" rpy="0 0 0"/>
+      <parent link="${namespace}/camera_${camera_suffix}_left_optical_link" />
+      <child link="${namespace}/camera_${camera_suffix}_right_optical_link" />
+    </joint>
+<gazebo reference="${namespace}/camera_${camera_suffix}_left_optical_link">
     <sensor type="multicamera" name="stereo_camera">
       <!-- see MultiSenseSLPlugin.h for available modes -->
