Commit message: switched to LPE

File: robot_description/noir_base.urdf (robot description, URDF)
Before this commit: robot noir, 11 links, 10 joints
Links:
- added link fcu
- added link fcu_frd
- added link laser_link, mass 1e-5
- link /camera_front_left_optical_link: geometry collision cylinder length=0.04 radius=0.04
- link /camera_front_right_optical_link: geometry collision cylinder length=0.04 radius=0.04
- link base_link_inertia: geometry collision box size=0.255 0.255 0.09; visual mesh filename=model://noir_description/meshes/CF_assembly.stl scale=1 1 1
Joints:
- added joint fcu_frd_joint: type fixed, parent fcu, child fcu_frd, origin xyz=0 0 0 rpy=3.14159265359 0 0
- added joint fcu_joint: type fixed, parent base_link, child fcu, origin xyz=0 0 0 rpy=0 0 0
- added joint laser_joint: type fixed, parent base_link, child laser_link, origin xyz=0.03 0.138 0.07 rpy=0 1.57079632679 0
- joint /camera_front_left_optical_joint: origin xyz=0 0 0.4 rpy=0 0 0 -> xyz=0.17 0.03805 0.01 rpy=0 0.78539816339 0
- joint /camera_front_right_optical_joint: origin xyz=0 -0.076 0 rpy=0 0 0 -> xyz=0 -0.0761 0 rpy=0 0 0

File: robot_description/noir_description/urdf/component_snippets.xacro (robot description, xacro)
@@ -30,4 +30,53 @@
         <rotorVelocitySlowdownSim>${rotor_velocity_slowdown_sim}</rotorVelocitySlowdownSim>
       </plugin>
+    </gazebo>
+  </xacro:macro>
+<!-- range sensor -->
+<xacro:macro name="sonar_sensor" params="name parent *origin ros_topic update_rate min_range max_range field_of_view ray_count">
+    <link name="${name}_link">
+      <inertial>
+        <mass value="1e-5" />
+        <origin xyz="0 0 0" rpy="0 0 0" />
+        <inertia ixx="1e-6" ixy="0" ixz="0" iyy="1e-6" iyz="0" izz="1e-6" />
+      </inertial>
+	</link>
+    <joint name="${name}_joint" type="fixed">
+      <xacro:insert_block name="origin" />
+      <parent link="${parent}"/>
+      <child link="${name}_link"/>
+    </joint>
+    <gazebo reference="${name}_link">
+      <sensor type="ray" name="${name}">
+        <always_on>true</always_on>
+        <update_rate>${update_rate}</update_rate>
+        <pose>0 0 0 0 0 0</pose>
+        <visualize>false</visualize>
+        <ray>
+          <scan>
+            <horizontal>
+              <samples>${ray_count}</samples>
+              <resolution>1</resolution>
+              <min_angle>-${field_of_view/2}</min_angle>
+              <max_angle> ${field_of_view/2}</max_angle>
+            </horizontal>
+            <vertical>
+              <samples>${ray_count}</samples>
+              <resolution>1</resolution>
+              <min_angle>-${field_of_view/2}</min_angle>
+              <max_angle> ${field_of_view/2}</max_angle>
+            </vertical>
+          </scan>
+          <range>
+            <min>${min_range}</min>
+            <max>${max_range}</max>
+            <resolution>0.01</resolution>
+          </range>
+        </ray>
+        <plugin name="gazebo_ros_${name}_controller" filename="libhector_gazebo_ros_sonar.so">
+          <gaussianNoise>0.005</gaussianNoise>
+          <topicName>${ros_topic}</topicName>
+          <frameId>${name}_link</frameId>
+        </plugin>
+      </sensor>
     </gazebo>
   </xacro:macro>

File: robot_description/noir_description/urdf/multirotor_base.xacro (robot description, xacro)
@@ -34,5 +34,5 @@
       </inertial>
       <visual>
-        <origin xyz="0 0 0" rpy="0 0 0" />
+        <origin xyz="0 0 0.052" rpy="0 0 0" />
         <geometry>
           <mesh filename="model://noir_description/meshes/${mesh_file}"

File: robot_description/noir_description/urdf/noir.xacro (robot description, xacro)
@@ -9,6 +9,6 @@
   <xacro:property name="mesh_scale_prop" value="1 1 1"/>
   <xacro:property name="mass" value="5" /> <!-- [kg] -->
-  <xacro:property name="body_width" value="1.05" /> <!-- [m] -->
-  <xacro:property name="body_height" value="0.20" /> <!-- [m] -->
+  <xacro:property name="body_width" value="0.255" /> <!-- [m] -->
+  <xacro:property name="body_height" value="0.09" /> <!-- [m] -->
   <xacro:property name="mass_rotor" value="0.05" /> <!-- [kg] -->
   <xacro:property name="arm_length_front_x" value="0.265" /> <!-- [m] -->

File: robot_description/noir_description/urdf/noir_base.xacro (robot description, xacro)
@@ -38,4 +38,17 @@
         />
   </xacro:if>
+<!-- Set up extra frames-->
+<link name="fcu"/>
+<joint name="fcu_joint" type="fixed">
+      <origin xyz="0 0 0" rpy="0 0 0" />
+      <parent link="base_link" />
+      <child link="fcu" />
+</joint>
+<link name="fcu_frd"/>
+<joint name="fcu_frd_joint" type="fixed">
+      <origin xyz="0 0 0" rpy="3.14159265359 0 0" />
+      <parent link="fcu" />
+      <child link="fcu_frd" />
+</joint>
 <!--stereo camera-->
 <xacro:if value="true">
@@ -44,11 +57,24 @@
     camera_suffix="front"
 parent_link="base_link"
-base_line="0.076"
-enable_visual="true"
+base_line="0.0761"
+enable_visual="false"
     >
 <cylinder length="0.04" radius="0.04" />
-    <origin xyz="0 0 0.4" rpy="0 0 0" />
+    <origin xyz="0.17 0.03805 0.01" rpy="0 0.78539816339 0" />
 </xacro:stereo_camera_macro>
 </xacro:if>
+<!--range sensor-->
+<xacro:sonar_sensor
+    name="laser"
+parent="base_link"
+ros_topic="/mavros/distance_sensor/laser_1_sub"
+update_rate="20"
+min_range="0.1"
+max_range="10"
+field_of_view="0.001"
+ray_count="1"
+>
+<origin xyz="0.03 0.138 0.07" rpy="0 1.57079632679 0" />
+</xacro:sonar_sensor>
 <!--standard camera-->
 <xacro:if value="false">
